Commit message: Update robot_3d_base.urdf.xacro

File: mec_mobile_description/urdf/mech/robot_3d_base.urdf.xacro (robot description, xacro)
@@ -4,5 +4,5 @@
 <xacro:property name="wheel_width" value="0.0304" />
 <xacro:property name="wheel_radius" value="0.0325" />
-<xacro:property name="total_height" value="0.26225" />
+<xacro:property name="total_height" value="0.17225" />
 <xacro:property name="base_length" value="0.300" />
 <xacro:property name="centered_length" value="0.238" />

Commit message: Update robot_3d_base.urdf.xacro

File: mec_mobile_description/urdf/mech/robot_3d_base.urdf.xacro (robot description, xacro)
@@ -4,5 +4,5 @@
 <xacro:property name="wheel_width" value="0.0304" />
 <xacro:property name="wheel_radius" value="0.0325" />
-<xacro:property name="total_height" value="0.26225" />
+<xacro:property name="total_height" value="0.16225" />
 <xacro:property name="base_length" value="0.300" />
 <xacro:property name="centered_length" value="0.238" />

Commit message: Update robot_3d_base.urdf.xacro

File: mec_mobile_description/urdf/mech/robot_3d_base.urdf.xacro (robot description, xacro)
@@ -4,5 +4,5 @@
 <xacro:property name="wheel_width" value="0.0304" />
 <xacro:property name="wheel_radius" value="0.0325" />
-<xacro:property name="total_height" value="0.17225" />
+<xacro:property name="total_height" value="0.16225" />
 <xacro:property name="base_length" value="0.300" />
 <xacro:property name="centered_length" value="0.238" />
