Commit message: Update robot_3d.urdf.xacro friction

File: mec_mobile_description/urdf/robots/robot_3d.urdf.xacro (robot description, xacro)
@@ -1,4 +1,4 @@
 <?xml version="1.0"?>
-<robot xmlns:xacro="http://www.ros.org/wiki/xacro" name="robot_3d">
+<robot name="robot_3d" xmlns:xacro="http://www.ros.org/wiki/xacro" xmlns:gz="http://gazebosim.org/schema">
     <xacro:property name="M_PI" value="3.1415926535897931" />
     <xacro:arg name="robot_name" default="robot_3d"/>
@@ -54,4 +54,62 @@
       update_rate="15.0"
       topic_name="imu/data"/>
+    <!-- Gazebo frictions -->
+  <gazebo reference='front_left_wheel'>
+    <collision>
+      <surface>
+        <friction>
+          <ode>
+            <mu>1.5</mu>
+            <mu2>0.0</mu2>
+            <fdir1 gz:expressed_in="base_footprint">1 -1 0</fdir1>
+          </ode>
+        </friction>
+      </surface>
+    </collision>
+  </gazebo>
+  <gazebo reference='back_left_wheel'>
+    <collision>
+      <surface>
+        <friction>
+          <ode>
+            <mu>1.5</mu>
+            <mu2>0.0</mu2>
+            <fdir1 gz:expressed_in="base_footprint">1 1 0</fdir1>
+          </ode>
+        </friction>
+      </surface>
+    </collision>
+  </gazebo>
+  <gazebo reference='front_right_wheel'>
+    <collision>
+      <surface>
+        <friction>
+          <ode>
+            <mu>1.5</mu>
+            <mu2>0.0</mu2>
+            <fdir1 gz:expressed_in="base_footprint">1 1 0</fdir1>
+          </ode>
+        </friction>
+      </surface>
+    </collision>
+  </gazebo>
+  <gazebo reference='back_right_wheel'>
+    <collision>
+      <surface>
+        <friction>
+          <ode>
+            <mu>1.5</mu>
+            <mu2>0.0</mu2>
+            <fdir1 gz:expressed_in="base_footprint">1 -1 0</fdir1>
+          </ode>
+        </friction>
+      </surface>
+    </collision>
+  </gazebo>
+  <gazebo reference="base_link">
+    <mu1>0.000002</mu1>
+    <mu2>0.000002</mu2>
+    <!-- <material>Gazebo/Red</material> -->
+  </gazebo>
     <!--
     <xacro:include filename="$(find mec_mobile_description)/urdf/control/velocity_control_plugin.urdf.xacro" />

Commit message: Update robot_3d.urdf.xacro

File: mec_mobile_description/urdf/robots/robot_3d.urdf.xacro (robot description, xacro)
@@ -54,5 +54,5 @@
       update_rate="15.0"
       topic_name="imu/data"/>
-  <!-- 6 - Gazebo frictions -->
+  <!-- 2.3 add Gazebo frictions -->
   <gazebo reference='front_left_wheel_link'>
     <collision>
@@ -112,3 +112,43 @@
     <!-- <material>Gazebo/Red</material> -->
   </gazebo>
+  <!-- 2.4 Camera physical properties -->
+  <joint type="fixed" name="camera_joint">
+    <origin xyz="0.1 0 0.06" rpy="0 0 0"/>
+    <child link="camera_link"/>
+    <parent link="base_link"/>
+    <axis xyz="0 1 0" />
+  </joint>
+  <link name='camera_link'>
+    <pose>0 0 0 0 0 0</pose>
+    <inertial>
+      <mass value="0.1"/>
+      <origin xyz="0 0 0" rpy="0 0 0"/>
+      <inertia
+          ixx="1e-6" ixy="0" ixz="0"
+          iyy="1e-6" iyz="0"
+          izz="1e-6"/>
+    </inertial>
+    <collision name='collision'>
+      <origin xyz="0 0 0" rpy="0 0 0"/>
+      <geometry>
+        <box size=".03 .03 .03"/>
+      </geometry>
+    </collision>
+    <visual name='camera_link_visual'>
+      <origin xyz="0 0 0" rpy="0 0 0"/>
+      <geometry>
+        <box size=".03 .03 .03"/>
+      </geometry>
+    </visual>
+  </link>
+  <gazebo reference="camera_link">
+    <material>Gazebo/Red</material>
+  </gazebo>
+  <joint type="fixed" name="camera_optical_joint">
+    <origin xyz="0 0 0" rpy="-1.5707 0 -1.5707"/>
+    <child link="camera_link_optical"/>
+    <parent link="camera_link"/>
+  </joint>
+  <link name="camera_link_optical">
+  </link>
 </robot>

Commit message: Update robot_3d.urdf.xacro

File: mec_mobile_description/urdf/robots/robot_3d.urdf.xacro (robot description, xacro)
@@ -7,5 +7,5 @@
     <xacro:include filename="$(find mec_mobile_description)/urdf/mech/robot_3d_base.urdf.xacro"/>
     <xacro:include filename="$(find mec_mobile_description)/urdf/mech/mecanum_wheel.urdf.xacro"/>
-    <xacro:include filename="$(find mec_mobile_description)/urdf/sensors/rgbd_camera.urdf.xacro"/>
+    <!-- <xacro:include filename="$(find mec_mobile_description)/urdf/sensors/rgbd_camera.urdf.xacro"/> -->
     <xacro:include filename="$(find mec_mobile_description)/urdf/sensors/lidar.urdf.xacro"/>
     <xacro:include filename="$(find mec_mobile_description)/urdf/sensors/imu.urdf.xacro"/>
@@ -32,9 +32,9 @@
       x_reflect="-1"
       y_reflect="-1"/>
-    <xacro:rgbd_camera
+    <!-- <xacro:rgbd_camera
       prefix="$(arg prefix)"
       camera_name="cam_1"
       xyz_offset="0.105 0 0.03"
-      rpy_offset="0 0 0"/>
+      rpy_offset="0 0 0"/> -->
     <xacro:lidar_sensor
       prefix="$(arg prefix)"
@@ -54,101 +54,101 @@
       update_rate="15.0"
       topic_name="imu/data"/>
-  <!-- 2.3 add Gazebo frictions -->
-  <gazebo reference='front_left_wheel_link'>
-    <collision>
-      <surface>
-        <friction>
-          <ode>
-            <mu>1.5</mu>
-            <mu2>0.0</mu2>
-            <fdir1 gz:expressed_in="base_footprint">1 -1 0</fdir1>
-          </ode>
-        </friction>
-      </surface>
-    </collision>
-  </gazebo>
-  <gazebo reference='back_left_wheel_link'>
-    <collision>
-      <surface>
-        <friction>
-          <ode>
-            <mu>1.5</mu>
-            <mu2>0.0</mu2>
-            <fdir1 gz:expressed_in="base_footprint">1 1 0</fdir1>
-          </ode>
-        </friction>
-      </surface>
-    </collision>
-  </gazebo>
-  <gazebo reference='front_right_wheel_link'>
-    <collision>
-      <surface>
-        <friction>
-          <ode>
-            <mu>1.5</mu>
-            <mu2>0.0</mu2>
-            <fdir1 gz:expressed_in="base_footprint">1 1 0</fdir1>
-          </ode>
-        </friction>
-      </surface>
-    </collision>
-  </gazebo>
-  <gazebo reference='back_right_wheel_link'>
-    <collision>
-      <surface>
-        <friction>
-          <ode>
-            <mu>1.5</mu>
-            <mu2>0.0</mu2>
-            <fdir1 gz:expressed_in="base_footprint">1 -1 0</fdir1>
-          </ode>
-        </friction>
-      </surface>
-    </collision>
-  </gazebo>
-  <gazebo reference="base_link">
-    <mu1>0.000002</mu1>
-    <mu2>0.000002</mu2>
-    <!-- <material>Gazebo/Red</material> -->
-  </gazebo>
-  <!-- 2.4 Camera physical properties -->
-  <joint type="fixed" name="camera_joint">
-    <origin xyz="0.1 0 0.06" rpy="0 0 0"/>
-    <child link="camera_link"/>
-    <parent link="base_link"/>
-    <axis xyz="0 1 0" />
-  </joint>
-  <link name='camera_link'>
-    <pose>0 0 0 0 0 0</pose>
-    <inertial>
-      <mass value="0.1"/>
-      <origin xyz="0 0 0" rpy="0 0 0"/>
-      <inertia
-          ixx="1e-6" ixy="0" ixz="0"
-          iyy="1e-6" iyz="0"
-          izz="1e-6"/>
-    </inertial>
-    <collision name='collision'>
-      <origin xyz="0 0 0" rpy="0 0 0"/>
-      <geometry>
-        <box size=".03 .03 .03"/>
-      </geometry>
-    </collision>
-    <visual name='camera_link_visual'>
-      <origin xyz="0 0 0" rpy="0 0 0"/>
-      <geometry>
-        <box size=".03 .03 .03"/>
-      </geometry>
-    </visual>
-  </link>
-  <gazebo reference="camera_link">
-    <material>Gazebo/Red</material>
-  </gazebo>
-  <joint type="fixed" name="camera_optical_joint">
-    <origin xyz="0 0 0" rpy="-1.5707 0 -1.5707"/>
-    <child link="camera_link_optical"/>
-    <parent link="camera_link"/>
-  </joint>
-  <link name="camera_link_optical">
-  </link>
+    <!-- 2.3 add Gazebo frictions -->
+    <gazebo reference='front_left_wheel_link'>
+      <collision>
+        <surface>
+          <friction>
+            <ode>
+              <mu>1.5</mu>
+              <mu2>0.0</mu2>
+              <fdir1 gz:expressed_in="base_footprint">1 -1 0</fdir1>
+            </ode>
+          </friction>
+        </surface>
+      </collision>
+    </gazebo>
+    <gazebo reference='back_left_wheel_link'>
+      <collision>
+        <surface>
+          <friction>
+            <ode>
+              <mu>1.5</mu>
+              <mu2>0.0</mu2>
+              <fdir1 gz:expressed_in="base_footprint">1 1 0</fdir1>
+            </ode>
+          </friction>
+        </surface>
+      </collision>
+    </gazebo>
+    <gazebo reference='front_right_wheel_link'>
+      <collision>
+        <surface>
+          <friction>
+            <ode>
+              <mu>1.5</mu>
+              <mu2>0.0</mu2>
+              <fdir1 gz:expressed_in="base_footprint">1 1 0</fdir1>
+            </ode>
+          </friction>
+        </surface>
+      </collision>
+    </gazebo>
+    <gazebo reference='back_right_wheel_link'>
+      <collision>
+        <surface>
+          <friction>
+            <ode>
+              <mu>1.5</mu>
+              <mu2>0.0</mu2>
+              <fdir1 gz:expressed_in="base_footprint">1 -1 0</fdir1>
+            </ode>
+          </friction>
+        </surface>
+      </collision>
+    </gazebo>
+    <gazebo reference="base_link">
+      <mu1>0.000002</mu1>
+      <mu2>0.000002</mu2>
+      <!-- <material>Gazebo/Red</material> -->
+    </gazebo>
+    <!-- 2.4.1 Camera physical properties -->
+    <joint type="fixed" name="camera_joint">
+      <origin xyz="0.1 0 0.04" rpy="0 0 0"/>
+      <child link="camera_link"/>
+      <parent link="base_link"/>
+      <axis xyz="0 1 0" />
+    </joint>
+    <link name='camera_link'>
+      <pose>0 0 0 0 0 0</pose>
+      <inertial>
+        <mass value="0.1"/>
+        <origin xyz="0 0 0" rpy="0 0 0"/>
+        <inertia
+            ixx="1e-6" ixy="0" ixz="0"
+            iyy="1e-6" iyz="0"
+            izz="1e-6"/>
+      </inertial>
+      <collision name='collision'>
+        <origin xyz="0 0 0" rpy="0 0 0"/>
+        <geometry>
+          <box size=".03 .03 .03"/>
+        </geometry>
+      </collision>
+      <visual name='camera_link_visual'>
+        <origin xyz="0 0 0" rpy="0 0 0"/>
+        <geometry>
+          <box size=".03 .03 .03"/>
+        </geometry>
+      </visual>
+    </link>
+    <gazebo reference="camera_link">
+      <material>Gazebo/Red</material>
+    </gazebo>
+    <joint type="fixed" name="camera_optical_joint">
+      <origin xyz="0 0 0" rpy="-1.5707 0 -1.5707"/>
+      <child link="camera_link_optical"/>
+      <parent link="camera_link"/>
+    </joint>
+    <link name="camera_link_optical">
+    </link>
 </robot>

Commit message: Update robot_3d.urdf.xacro

File: mec_mobile_description/urdf/robots/robot_3d.urdf.xacro (robot description, xacro)
@@ -114,5 +114,5 @@
     <!-- 2.5.1 Camera physical properties -->
     <joint type="fixed" name="camera_joint">
-      <origin xyz="0.1 0 0.04" rpy="0 0 0"/>
+      <origin xyz="0.092 0 0.05" rpy="0 0 0"/>
       <child link="camera_link"/>
       <parent link="base_link"/>
@@ -138,5 +138,5 @@
         <origin xyz="0 0 0" rpy="0 0 0"/>
         <geometry>
-          <box size=".03 .03 .03"/>
+          <box size=".02 .02 .02"/>
         </geometry>
       </visual>
